Commit message: Imported upstream version '1.0.5' of 'upstream'

File: uol_turtlebot_simulator/urdf/kobuki_hexagons_kinect.urdf.xacro (robot description, xacro)
@@ -6,5 +6,8 @@
 -->
 <robot name="turtlebot" xmlns:xacro="http://ros.org/wiki/xacro">
-  <xacro:include filename="$(find uol_turtlebot_simulator)/urdf/turtlebot_library.urdf.xacro" />
+  <xacro:include filename="$(find turtlebot_description)/urdf/turtlebot_common_library.urdf.xacro" />
+  <xacro:include filename="$(find kobuki_description)/urdf/kobuki.urdf.xacro" />
+  <xacro:include filename="$(find turtlebot_description)/urdf/stacks/hexagons.urdf.xacro"/>
+  <xacro:include filename="$(find uol_turtlebot_simulator)/urdf/sensors/kinect.urdf.xacro"/>
   <kobuki/>
   <stack_hexagons parent="base_link"/>

File: uol_turtlebot_simulator/urdf/sensors/kinect.urdf.xacro (robot description, xacro)
@@ -2,21 +2,14 @@
 <robot name="sensor_kinect" xmlns:xacro="http://ros.org/wiki/xacro">
   <xacro:include filename="$(find uol_turtlebot_simulator)/urdf/turtlebot_gazebo.urdf.xacro"/>
-  <xacro:include filename="$(find uol_turtlebot_simulator)/urdf/turtlebot_properties.urdf.xacro"/>
+  <xacro:include filename="$(find turtlebot_description)/urdf/turtlebot_properties.urdf.xacro"/>
+  <xacro:property name="kinect_cam_py" value="-0.0125"/>
   <!-- Parameterised in part by the values in turtlebot_properties.urdf.xacro -->
   <xacro:macro name="sensor_kinect" params="parent">
     <joint name="camera_rgb_joint" type="fixed">
-      <origin xyz="${cam_px} ${cam_py} ${cam_pz}" rpy="${cam_or} ${cam_op} ${cam_oy}"/>
+      <origin xyz="${cam_px} ${kinect_cam_py} ${cam_pz}" rpy="${cam_or} ${cam_op} ${cam_oy}"/>
       <parent link="${parent}"/>
       <child link="camera_rgb_frame" />
     </joint>
-    <link name="camera_rgb_frame">
-      <inertial>
-        <mass value="0.001" />
-        <origin xyz="0 0 0" />
-        <inertia ixx="0.0001" ixy="0.0" ixz="0.0"
-                 iyy="0.0001" iyz="0.0"
-                 izz="0.0001" />
-      </inertial>
-    </link>
+    <link name="camera_rgb_frame"/>
     <joint name="camera_rgb_optical_joint" type="fixed">
       <origin xyz="0 0 0" rpy="${-M_PI/2} 0 ${-M_PI/2}" />
@@ -24,56 +17,40 @@
       <child link="camera_rgb_optical_frame" />
     </joint>
-    <link name="camera_rgb_optical_frame">
+    <link name="camera_rgb_optical_frame"/>
+    <joint name="camera_joint" type="fixed">
+      <origin xyz="-0.031 ${-kinect_cam_py} -0.016" rpy="0 0 0"/>
+      <parent link="camera_rgb_frame"/>
+      <child link="camera_link"/>
+    </joint>
+      <link name="camera_link">
+      <visual>
+       <origin xyz="0 0 0" rpy="0 0 ${M_PI/2}"/>
+        <geometry>
+         <mesh filename="package://turtlebot_description/meshes/sensors/kinect.dae"/>
+        </geometry>
+      </visual>
+  	  <collision>
+        <origin xyz="0.0 0.0 0.0" rpy="0 0 0"/>
+  	    <geometry>
+  	      <box size="0.07271 0.27794 0.073"/>
+  	    </geometry>
+  	  </collision>
       <inertial>
-        <mass value="0.001" />
+        <mass value="0.564" />
         <origin xyz="0 0 0" />
-        <inertia ixx="0.0001" ixy="0.0" ixz="0.0"
-                 iyy="0.0001" iyz="0.0"
-                 izz="0.0001" />
+        <inertia ixx="0.003881243" ixy="0.0" ixz="0.0"
+                 iyy="0.000498940" iyz="0.0"
+                 izz="0.003879257" />
       </inertial>
     </link>
-  <joint name="camera_joint" type="fixed">
-    <origin xyz="-0.031 ${-cam_py} -0.016" rpy="0 0 0"/>
-    <parent link="camera_rgb_frame"/>
-    <child link="camera_link"/>
-  </joint>
-    <link name="camera_link">
-    <visual>
-     <origin xyz="0 0 0" rpy="0 0 ${M_PI/2}"/>
-      <geometry>
-       <mesh filename="package://uol_turtlebot_simulator/meshes/sensors/kinect.dae"/>
-      </geometry>
-    </visual>
-	  <collision>
-      <origin xyz="0.0 0.0 0.0" rpy="0 0 0"/>
-	    <geometry>
-	      <box size="0.07271 0.27794 0.073"/>
-	    </geometry>
-	  </collision>
-    <inertial>
-      <mass value="0.001" />
-      <origin xyz="0 0 0" />
-      <inertia ixx="0.0001" ixy="0.0" ixz="0.0"
-               iyy="0.0001" iyz="0.0"
-               izz="0.0001" />
-    </inertial>
-  </link>
-  <!-- The fixed joints & links below are usually published by static_transformers launched by the OpenNi launch
-       files. However, for Gazebo simulation we need them, so we add them here.
-       (Hence, don't publish them additionally!) -->
+    <!-- The fixed joints & links below are usually published by static_transformers launched by the OpenNi launch
+         files. However, for Gazebo simulation we need them, so we add them here.
+         (Hence, don't publish them additionally!) -->
 	<joint name="camera_depth_joint" type="fixed">
-	  <origin xyz="0 ${2 * -cam_py} 0" rpy="0 0 0" />
+	  <origin xyz="0 ${2 * -kinect_cam_py} 0" rpy="0 0 0" />
 	  <parent link="camera_rgb_frame" />
 	  <child link="camera_depth_frame" />
 	</joint>
-	<link name="camera_depth_frame">
-    <inertial>
-      <mass value="0.001" />
-      <origin xyz="0 0 0" />
-      <inertia ixx="0.0001" ixy="0.0" ixz="0.0"
-               iyy="0.0001" iyz="0.0"
-               izz="0.0001" />
-    </inertial>
-	</link>
+	<link name="camera_depth_frame"/>
 	<joint name="camera_depth_optical_joint" type="fixed">
 	  <origin xyz="0 0 0" rpy="${-M_PI/2} 0 ${-M_PI/2}" />
@@ -81,13 +58,5 @@
 	  <child link="camera_depth_optical_frame" />
 	</joint>
-	<link name="camera_depth_optical_frame">
-    <inertial>
-      <mass value="0.001" />
-      <origin xyz="0 0 0" />
-      <inertia ixx="0.0001" ixy="0.0" ixz="0.0"
-               iyy="0.0001" iyz="0.0"
-               izz="0.0001" />
-    </inertial>
-	</link>
+	<link name="camera_depth_optical_frame"/>
 	<!-- Kinect sensor for simulation -->
 	<turtlebot_sim_3dsensor/>

File: uol_turtlebot_simulator/urdf/turtlebot_gazebo.urdf.xacro (robot description, xacro)
@@ -8,5 +8,5 @@
         <update_rate>20.0</update_rate>
         <camera>
-          <horizontal_fov>${60.0*M_PI/180.0}</horizontal_fov>
+          <horizontal_fov>${$(arg fov)*M_PI/180.0}</horizontal_fov>
           <image>
             <format>R8G8B8</format>
@@ -16,5 +16,5 @@
           <clip>
             <near>0.05</near>
-            <far>8.0</far>
+            <far>100.0</far>
           </clip>
         </camera>
@@ -35,6 +35,6 @@
           <distortion_t1>0.0</distortion_t1>
           <distortion_t2>0.0</distortion_t2>
-          <pointCloudCutoff>0.4</pointCloudCutoff>
-          <pointCloudCutoffMax>20</pointCloudCutoffMax>
+          <pointCloudCutoff>0.295</pointCloudCutoff>
+          <pointCloudCutoffMax>100</pointCloudCutoffMax>
         </plugin>
       </sensor>
